Commit message: slowly trying to fix the URDF manually, will be reexported from solidworks with fixed angle

File: robotURDF/urdf/000_Assy_Full.SLDASM.urdf (robot description, URDF)
Before this commit: robot 000_Assy_Full.SLDASM, 15 links, 13 joints
Links:
- removed link Four Bar Beam Right
- removed link Four Bar Link Right
